File: C-13X-PCB.sch (KiCad schematic (older format))
At the start: 20 parts, among them J1 ai03_Daughterboard_Connector, J2 AVR-TagConnect, SW1 SW_Push, SW2 SW_Push, U1 ATmega32A-AU, U2 SRV05-4, Y1 Crystal_GND24_Small

Commit message: Add LCSC part numbers in BOM, fix RGB
Parts:
- C1, C2: LCSC (none) -> C1653
- C3, C4: LCSC (none) -> C14663
- C5: LCSC (none) -> C15850
- D1, D2: LCSC (none) -> C2891771
- F1: LCSC (none) -> C69688
- J1: LCSC (none) -> C160404
- SW1, SW2: LCSC (none) -> C318884
- U1: LCSC (none) -> C5659
- U2: LCSC (none) -> C85364
- Y1: LCSC (none) -> C13738
Changed lines of the file:
@@
 F 2 "Diode_SMD:D_SOD-123" V 3800 2000 50  0001 C CNN
 F 3 "~" V 3800 2000 50  0001 C CNN
+F 4 "C2891771" H 3800 2000 50  0001 C CNN "LCSC"
 	1    3800 2000
 	0    -1   1    0
@@
 F 2 "Diode_SMD:D_SOD-123" V 3950 2000 50  0001 C CNN
 F 3 "~" V 3950 2000 50  0001 C CNN
+F 4 "C2891771" H 3950 2000 50  0001 C CNN "LCSC"
 	1    3950 2000
 	0    1    1    0
@@
 F 2 "Capacitor_SMD:C_0603_1608Metric" H 1100 6300 50  0001 C CNN
 F 3 "~" H 1100 6300 50  0001 C CNN
+F 4 "C14663" H 1100 6300 50  0001 C CNN "LCSC"
 	1    1100 6300
 	1    0    0    -1
@@
 F 2 "Capacitor_SMD:C_0603_1608Metric" H 1550 6300 50  0001 C CNN
 F 3 "~" H 1550 6300 50  0001 C CNN
+F 4 "C14663" H 1550 6300 50  0001 C CNN "LCSC"
 	1    1550 6300
 	1    0    0    -1
@@
 F 2 "Capacitor_SMD:C_0805_2012Metric" H 2000 6300 50  0001 C CNN
 F 3 "~" H 2000 6300 50  0001 C CNN
+F 4 "C15850" H 2000 6300 50  0001 C CNN "LCSC"
 	1    2000 6300
 	1    0    0    -1
@@
 F 2 "Capacitor_SMD:C_0603_1608Metric" H 7300 2250 50  0001 C CNN
 F 3 "~" H 7300 2250 50  0001 C CNN
+F 4 "C1653" H 7300 2250 50  0001 C CNN "LCSC"
 	1    7300 2250
 	0    -1   -1   0
@@
 F 2 "Capacitor_SMD:C_0603_1608Metric" H 7300 2550 50  0001 C CNN
 F 3 "~" H 7300 2550 50  0001 C CNN
+F 4 "C1653" H 7300 2550 50  0001 C CNN "LCSC"
 	1    7300 2550
 	0    -1   -1   0
@@
 F 2 "Button_Switch_SMD:SW_SPST_TL3342" H 7950 1850 50  0001 C CNN
 F 3 "~" H 7950 1850 50  0001 C CNN
+F 4 "C318884" H 7950 1650 50  0001 C CNN "LCSC"
 	1    7950 1650
 	1    0    0    -1
@@
 F 2 "Button_Switch_SMD:SW_SPST_TL3342" H 10500 5400 50  0001 C CNN
 F 3 "~" H 10500 5400 50  0001 C CNN
+F 4 "C318884" H 10500 5200 50  0001 C CNN "LCSC"
 	1    10500 5200
 	-1   0    0    -1
@@
 F 2 "Fuse:Fuse_1206_3216Metric_Pad1.42x1.75mm_HandSolder" V 1930 1450 50  0001 C CNN
 F 3 "~" H 2000 1450 50  0001 C CNN
+F 4 "C69688" H 2000 1450 50  0001 C CNN "LCSC"
 	1    2000 1450
 	0    1    1    0
@@
 F 2 "Connector_JST:JST_SH_SM04B-SRSS-TB_1x04-1MP_P1.00mm_Horizontal" H 1600 1150 50  0001 C CNN
 F 3 "~" H 1500 1550 50  0001 C CNN
+F 4 "C160404" H 1500 1550 50  0001 C CNN "LCSC"
 	1    1500 1550
 	-1   0    0    -1
@@
 F 2 "Package_QFP:TQFP-44_10x10mm_P0.8mm" H 8900 3800 50  0001 C CIN
 F 3 "http://ww1.microchip.com/downloads/en/DeviceDoc/atmel-8155-8-bit-microcontroller-avr-atmega32a_datasheet.pdf" H 8900 3800 50  0001 C CNN
+F 4 "C5659" H 8900 3800 50  0001 C CNN "LCSC"
 	1    8900 3800
 	1    0    0    -1
@@
 F 2 "Crystal:Crystal_SMD_3225-4Pin_3.2x2.5mm" H 7700 2400 50  0001 C CNN
 F 3 "~" H 7700 2400 50  0001 C CNN
+F 4 "C13738" H 7700 2400 50  0001 C CNN "LCSC"
 	1    7700 2400
 	0    1    1    0
@@
 F 2 "Package_TO_SOT_SMD:SOT-23-6" H 3650 1150 50  0001 C CNN
 F 3 "http://www.onsemi.com/pub/Collateral/SRV05-4-D.PDF" H 2950 1600 50  0001 C CNN
+F 4 "C85364" H 2950 1600 50  0001 C CNN "LCSC"
 	1    2950 1600
 	0    1    -1   0
